File: Hardware/Main_Board/SD_Storage.sch (KiCad schematic (older format))
At the start: 3 parts

Commit message: [HARDWARE] Component association + schematic modifications
Parts:
- removed U?: SD_HOLDER, symbol SD_HOLDER
- added U6: MICROSD_HOLDER, symbol MICROSD_HOLDER
- gave numbers to parts that had none: 2
Connections:
- wire segments 15 -> 14
- no-connect marks 1 -> 2
Changed lines of the file:
@@
-EESchema Schematic File Version 2  date jeu. 10 oct. 2013 13:52:33 CEST
+EESchema Schematic File Version 2  date mer. 16 oct. 2013 19:37:53 CEST
 LIBS:power
 LIBS:device
@@
 LIBS:ap1117
 LIBS:l298
+LIBS:conn_4_jst
+LIBS:conn_2_jst
+LIBS:microsd_holder
 LIBS:ausbee-cache
 EELAYER 25  0
@@
 Sheet 5 6
 Title ""
-Date "10 oct 2013"
+Date "16 oct 2013"
 Rev ""
 Comp ""
@@
 $EndDescr
 Wire Wire Line
+	4000 3350 4400 3350
+Wire Wire Line
+	4400 3150 4350 3150
+Wire Wire Line
 	6600 3750 6600 3800
 Wire Wire Line
@@
 	4350 3650 4400 3650
 Wire Wire Line
-	4400 3150 4350 3150
-Wire Wire Line
 	4400 3550 4350 3550
 Wire Wire Line
 	4350 3550 4350 3600
-Wire Wire Line
-	4400 3250 4350 3250
-Wire Wire Line
-	4350 3250 4350 3300
-Wire Wire Line
-	4400 3350 4200 3350
 Wire Wire Line
 	4350 4100 4350 4050
@@
 	4350 3450 4400 3450
 Wire Wire Line
-	4350 3050 4400 3050
-Wire Wire Line
 	4400 3950 3700 3950
 Connection ~ 3850 3950
 Wire Wire Line
 	6600 3350 6600 3300
+Wire Wire Line
+	5450 4450 5450 4400
+Wire Wire Line
+	4350 3250 4400 3250
+NoConn ~ 4400 3050
+Text HLabel 4350 3150 0    60   Input ~ 0
+SS
 $Comp
-L GND #PWR?
+L GND #PWR147
+U 1 1 525ECE80
+P 5450 4450
+F 0 "#PWR147" H 5450 4450 30  0001 C CNN
+F 1 "GND" H 5450 4380 30  0001 C CNN
+	1    5450 4450
+	1    0    0    -1
+$EndComp
+$Comp
+L MICROSD_HOLDER U6
+U 1 1 525ECE5E
+P 5400 3600
+F 0 "U6" H 5950 3000 60  0000 C CNN
+F 1 "MICROSD_HOLDER" H 5600 3700 60  0000 C CNN
+	1    5400 3600
+	1    0    0    -1
+$EndComp
+$Comp
+L GND #PWR149
 U 1 1 525142D2
 P 6600 3800
-F 0 "#PWR?" H 6600 3800 30  0001 C CNN
+F 0 "#PWR149" H 6600 3800 30  0001 C CNN
 F 1 "GND" H 6600 3730 30  0001 C CNN
 	1    6600 3800
@@
 $EndComp
 $Comp
-L +3.3V #PWR?
+L +3.3V #PWR148
 U 1 1 525142CF
 P 6600 3300
-F 0 "#PWR?" H 6600 3260 30  0001 C CNN
+F 0 "#PWR148" H 6600 3260 30  0001 C CNN
 F 1 "+3.3V" H 6600 3410 30  0000 C CNN
 	1    6600 3300
@@
 $EndComp
 $Comp
-L C C?
+L C C34
 U 1 1 525142CB
 P 6600 3550
-F 0 "C?" H 6650 3650 50  0000 L CNN
+F 0 "C34" H 6650 3650 50  0000 L CNN
 F 1 "100n" H 6650 3450 50  0000 L CNN
 	1    6600 3550
@@
 $EndComp
 $Comp
-L +3.3V #PWR?
+L +3.3V #PWR143
 U 1 1 525142AE
 P 3850 3400
-F 0 "#PWR?" H 3850 3360 30  0001 C CNN
+F 0 "#PWR143" H 3850 3360 30  0001 C CNN
 F 1 "+3.3V" H 3850 3510 30  0000 C CNN
 	1    3850 3400
@@
 $EndComp
 $Comp
-L R R?
+L R R10
 U 1 1 525142AC
 P 3850 3700
-F 0 "R?" V 3930 3700 50  0000 C CNN
+F 0 "R10" V 3930 3700 50  0000 C CNN
 F 1 "10k" V 3850 3700 50  0000 C CNN
 	1    3850 3700
@@
 $EndComp
 $Comp
-L GND #PWR?
+L GND #PWR146
 U 1 1 5251424F
 P 4350 4100
-F 0 "#PWR?" H 4350 4100 30  0001 C CNN
+F 0 "#PWR146" H 4350 4100 30  0001 C CNN
 F 1 "GND" H 4350 4030 30  0001 C CNN
 	1    4350 4100
@@
 $EndComp
 $Comp
-L GND #PWR?
+L GND #PWR145
 U 1 1 52514242
 P 4350 3600
-F 0 "#PWR?" H 4350 3600 30  0001 C CNN
+F 0 "#PWR145" H 4350 3600 30  0001 C CNN
 F 1 "GND" H 4350 3530 30  0001 C CNN
 	1    4350 3600
@@
 $EndComp
 $Comp
-L +3.3V #PWR?
+L +3.3V #PWR144
 U 1 1 52514239
-P 4200 3350
-F 0 "#PWR?" H 4200 3310 30  0001 C CNN
-F 1 "+3.3V" H 4200 3460 30  0000 C CNN
-	1    4200 3350
-	1    0    0    -1
-$EndComp
-$Comp
-L GND #PWR?
-U 1 1 5251422F
-P 4350 3300
-F 0 "#PWR?" H 4350 3300 30  0001 C CNN
-F 1 "GND" H 4350 3230 30  0001 C CNN
-	1    4350 3300
+P 4000 3350
+F 0 "#PWR144" H 4000 3310 30  0001 C CNN
+F 1 "+3.3V" H 4000 3460 30  0000 C CNN
+	1    4000 3350
 	1    0    0    -1
 $EndComp
@@
 Text HLabel 4350 3450 0    60   Input ~ 0
 SCK
-Text HLabel 4350 3150 0    60   Input ~ 0
+Text HLabel 4350 3250 0    60   Input ~ 0
 MOSI
-Text HLabel 4350 3050 0    60   Input ~ 0
-SS
-$Comp
-L SD_HOLDER U?
-U 1 1 525141A0
-P 5400 3600
-F 0 "U?" H 5950 3000 60  0000 C CNN
-F 1 "SD_HOLDER" H 5600 3700 60  0000 C CNN
-	1    5400 3600
-	1    0    0    -1
-$EndComp
 $EndSCHEMATC
