File: Hardware/Main_Board/power.sch (KiCad schematic (older format))
At the start: 10 parts, among them P17 CONN_2, P18 CONN_2, P19 CONN_2, P20 CONN_2, U4 AP1117, U5 AP1117

Commit message: [HARDWARE] Update schematic and start routing
Parts:
- added D17: LED, symbol LED
- added R20: 820, symbol R
Connections:
- net +5V: now also R20.1
- net GND: now also D17.2 (K)
- new net: D17.1 (A), R20.2
Changed lines of the file:
@@
-EESchema Schematic File Version 2  date mer. 16 oct. 2013 19:37:53 CEST
+EESchema Schematic File Version 2  date dim. 20 oct. 2013 18:50:44 CEST
 LIBS:power
 LIBS:device
@@
 Sheet 4 6
 Title ""
-Date "16 oct 2013"
+Date "20 oct 2013"
 Rev ""
 Comp ""
@@
 Comment4 ""
 $EndDescr
+Wire Wire Line
+	8850 2750 8850 2700
+Wire Wire Line
+	8850 3750 8850 3700
+Connection ~ 4300 3300
+Wire Wire Line
+	3950 3300 5550 3300
+Wire Wire Line
+	3950 3300 3950 3150
+Wire Wire Line
+	6850 4800 6800 4800
+Wire Wire Line
+	6850 5050 6850 5000
+Wire Wire Line
+	6850 5000 6800 5000
+Connection ~ 4900 3300
+Wire Wire Line
+	4300 3300 4300 3250
+Wire Wire Line
+	5550 2850 5550 2800
+Wire Wire Line
+	5550 2800 5500 2800
+Wire Wire Line
+	4900 3300 4900 3350
+Wire Wire Line
+	5550 3300 5550 3250
+Wire Wire Line
+	4300 2850 4300 2800
+Wire Wire Line
+	4800 5000 4850 5000
+Wire Wire Line
+	4850 5000 4850 5050
+Wire Wire Line
+	4850 4800 4800 4800
+Wire Wire Line
+	3150 4800 3100 4800
+Wire Wire Line
+	6250 2850 6250 2800
+Wire Wire Line
+	7500 3250 7500 3300
+Wire Wire Line
+	6850 3300 6850 3350
+Wire Wire Line
+	7500 2800 7500 2850
+Wire Wire Line
+	7500 3300 6250 3300
+Wire Wire Line
+	6250 3300 6250 3250
+Connection ~ 6850 3300
+Wire Wire Line
+	3150 5050 3150 5000
+Wire Wire Line
+	3150 5000 3100 5000
+Wire Wire Line
+	3950 2950 3950 2800
+Wire Wire Line
+	3950 2800 4300 2800
+Wire Wire Line
+	7650 2800 7450 2800
+Connection ~ 7500 2800
+Wire Wire Line
+	8850 3300 8850 3250
+$Comp
+L GND #PWR137
+U 1 1 52613E4B
+P 8850 3750
+F 0 "#PWR137" H 8850 3750 30  0001 C CNN
+F 1 "GND" H 8850 3680 30  0001 C CNN
+	1    8850 3750
+	1    0    0    -1
+$EndComp
+$Comp
+L LED D17
+U 1 1 52613E43
+P 8850 3500
+F 0 "D17" H 8850 3600 50  0000 C CNN
+F 1 "LED" H 8850 3400 50  0000 C CNN
+	1    8850 3500
+	0    1    1    0
+$EndComp
+$Comp
+L R R20
+U 1 1 52613E38
+P 8850 3000
+F 0 "R20" V 8930 3000 50  0000 C CNN
+F 1 "820" V 8850 3000 50  0000 C CNN
+	1    8850 3000
+	1    0    0    -1
+$EndComp
+$Comp
+L +5V #PWR136
+U 1 1 52613E32
+P 8850 2700
+F 0 "#PWR136" H 8850 2790 20  0001 C CNN
+F 1 "+5V" H 8850 2790 30  0000 C CNN
+	1    8850 2700
+	1    0    0    -1
+$EndComp
+$Comp
+L VDD #PWR135
+U 1 1 526131E7
+P 7650 2800
+F 0 "#PWR135" H 7650 2900 30  0001 C CNN
+F 1 "VDD" H 7650 2910 30  0000 C CNN
+	1    7650 2800
+	1    0    0    -1
+$EndComp
 $Comp
 L CP C33
@@
 	1    0    0    -1
 $EndComp
-Connection ~ 4300 3300
-Wire Wire Line
-	3950 3300 5550 3300
-Wire Wire Line
-	3950 3300 3950 3150
-Wire Wire Line
-	6850 4800 6800 4800
-Wire Wire Line
-	6850 5050 6850 5000
-Wire Wire Line
-	6850 5000 6800 5000
-Connection ~ 4900 3300
-Wire Wire Line
-	4300 3300 4300 3250
-Wire Wire Line
-	5550 2850 5550 2800
-Wire Wire Line
-	5550 2800 5500 2800
-Wire Wire Line
-	4900 3300 4900 3350
-Wire Wire Line
-	5550 3300 5550 3250
-Wire Wire Line
-	4300 2850 4300 2800
-Wire Wire Line
-	4800 5000 4850 5000
-Wire Wire Line
-	4850 5000 4850 5050
-Wire Wire Line
-	4850 4800 4800 4800
-Wire Wire Line
-	3150 4800 3100 4800
-Wire Wire Line
-	6250 2850 6250 2800
-Wire Wire Line
-	7500 3250 7500 3300
-Wire Wire Line
-	6850 3300 6850 3350
-Wire Wire Line
-	7450 2800 7500 2800
-Wire Wire Line
-	7500 2800 7500 2850
-Wire Wire Line
-	7500 3300 6250 3300
-Wire Wire Line
-	6250 3300 6250 3250
-Connection ~ 6850 3300
-Wire Wire Line
-	3150 5050 3150 5000
-Wire Wire Line
-	3150 5000 3100 5000
-Wire Wire Line
-	3950 2950 3950 2800
-Wire Wire Line
-	3950 2800 4300 2800
 $Comp
 L CONN_2 P18
@@
 MOTOR_POWER
 $Comp
-L GND #PWR141
+L GND #PWR133
 U 1 1 52558D99
 P 6850 5050
-F 0 "#PWR141" H 6850 5050 30  0001 C CNN
+F 0 "#PWR133" H 6850 5050 30  0001 C CNN
 F 1 "GND" H 6850 4980 30  0001 C CNN
 	1    6850 5050
@@
 $EndComp
 $Comp
-L +5V #PWR139
+L +5V #PWR131
 U 1 1 52553DBF
 P 6250 2800
-F 0 "#PWR139" H 6250 2890 20  0001 C CNN
+F 0 "#PWR131" H 6250 2890 20  0001 C CNN
 F 1 "+5V" H 6250 2890 30  0000 C CNN
 	1    6250 2800
@@
 $EndComp
 $Comp
-L +5V #PWR138
+L +5V #PWR130
 U 1 1 52553DB8
 P 5550 2800
-F 0 "#PWR138" H 5550 2890 20  0001 C CNN
+F 0 "#PWR130" H 5550 2890 20  0001 C CNN
 F 1 "+5V" H 5550 2890 30  0000 C CNN
 	1    5550 2800
@@
 $EndComp
 $Comp
-L GND #PWR137
+L GND #PWR129
 U 1 1 52553DB4
 P 4900 3350
-F 0 "#PWR137" H 4900 3350 30  0001 C CNN
+F 0 "#PWR129" H 4900 3350 30  0001 C CNN
 F 1 "GND" H 4900 3280 30  0001 C CNN
 	1    4900 3350
@@
 $EndComp
 $Comp
-L GND #PWR136
+L GND #PWR128
 U 1 1 52543C3B
 P 4850 5050
-F 0 "#PWR136" H 4850 5050 30  0001 C CNN
+F 0 "#PWR128" H 4850 5050 30  0001 C CNN
 F 1 "GND" H 4850 4980 30  0001 C CNN
 	1    4850 5050
@@
 AX12_POWER
 $Comp
-L GND #PWR135
+L GND #PWR127
 U 1 1 525198A8
 P 3150 5050
-F 0 "#PWR135" H 3150 5050 30  0001 C CNN
+F 0 "#PWR127" H 3150 5050 30  0001 C CNN
 F 1 "GND" H 3150 4980 30  0001 C CNN
 	1    3150 5050
@@
 3.3V regulator
 $Comp
-L GND #PWR140
+L GND #PWR132
 U 1 1 52516AEA
 P 6850 3350
-F 0 "#PWR140" H 6850 3350 30  0001 C CNN
+F 0 "#PWR132" H 6850 3350 30  0001 C CNN
 F 1 "GND" H 6850 3280 30  0001 C CNN
 	1    6850 3350
@@
 $EndComp
 $Comp
-L +3.3V #PWR142
+L +3.3V #PWR134
 U 1 1 52516ADF
 P 7500 2800
-F 0 "#PWR142" H 7500 2760 30  0001 C CNN
+F 0 "#PWR134" H 7500 2760 30  0001 C CNN
 F 1 "+3.3V" H 7500 2910 30  0000 C CNN
 	1    7500 2800
